File: doorbell.brd (EAGLE design)
At the start: 33 x 33 mm, 12 parts, among them Q1 8050

Commit message: Artwork + Board All Layers enabled
Parts:
- IC1: value (none) -> RTS-933-9A
Changed lines of the file:
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@@
 <attribute name="NAME" x="27.9292875" y="54.339409375" size="1.27" layer="25" ratio="10" rot="R225"/>
 </element>
-<element name="IC1" library="ic-package" library_urn="urn:adsk.eagle:library:239" package="SOCKET-16" package3d_urn="urn:adsk.eagle:package:14441/1" value="" x="28.79" y="44.3" smashed="yes">
+<element name="IC1" library="ic-package" library_urn="urn:adsk.eagle:library:239" package="SOCKET-16" package3d_urn="urn:adsk.eagle:package:14441/1" value="RTS-933-9A" x="28.79" y="44.3" smashed="yes">
 <attribute name="NAME" x="24.153" y="43.376" size="1.27" layer="25" ratio="10" rot="R180"/>
-<attribute name="VALUE" x="22.44" y="43.665" size="1.27" layer="27" ratio="10"/>
 </element>
 <element name="JP1" library="pinhead" library_urn="urn:adsk.eagle:library:325" package="1X02" package3d_urn="urn:adsk.eagle:package:22435/2" value="3V Battery" x="40.14" y="55.73" smashed="yes" rot="R270">
